Commit message: Added gazebo support to diff bot

File: src/differential_drive/src/description/ros2_control/diffbot.ros2_control.xacro (robot description, xacro)
@@ -1,7 +1,7 @@
 <?xml version="1.0"?>
 <robot xmlns:xacro="http://www.ros.org/wiki/xacro">
-  <xacro:macro name="diffbot_ros2_control" params="name prefix use_mock_hardware">
+  <xacro:macro name="diffbot_ros2_control" params="name prefix use_mock_hardware use_sim">
     <ros2_control name="${name}" type="system">
-      <xacro:unless value="${use_mock_hardware}">
+      <xacro:unless value="${use_mock_hardware or use_sim}">
         <hardware>
           <plugin>differential_drive_controller/DiffBotSystemHardware</plugin>
@@ -12,19 +12,37 @@
       <xacro:if value="${use_mock_hardware}">
         <hardware>
-          <plugin>mock_components/GenericSystem</plugin>
+          <plugin>mock_components/GenericSystem</plugin> [cite: 5]
           <param name="calculate_dynamics">true</param>
         </hardware>
       </xacro:if>
+      <xacro:if value="${use_sim}">
+        <hardware>
+          <plugin>gz_ros2_control/GazeboSimSystem</plugin>
+        </hardware>
+      </xacro:if>
       <joint name="${prefix}left_wheel_joint">
-        <command_interface name="velocity"/>
+        <command_interface name="velocity">
+            <param name="min">-10</param>
+            <param name="max">10</param>
+        </command_interface>
         <state_interface name="position"/>
         <state_interface name="velocity"/>
       </joint>
       <joint name="${prefix}right_wheel_joint">
-        <command_interface name="velocity"/>
+        <command_interface name="velocity">
+            <param name="min">-10</param>
+            <param name="max">10</param>
+        </command_interface>
         <state_interface name="position"/>
         <state_interface name="velocity"/>
       </joint>
     </ros2_control>
+    <xacro:if value="${use_sim}">
+      <gazebo>
+        <plugin filename="gz_ros2_control-system" name="gz_ros2_control::GazeboSimROS2ControlPlugin">
+          <parameters>$(find differential_drive_controller)/bringup/config/diffbot_controllers.yaml</parameters>
+        </plugin>
+      </gazebo>
+    </xacro:if>
   </xacro:macro>
 </robot>

File: src/differential_drive/src/description/urdf/diffbot.urdf.xacro (robot description, xacro)
@@ -4,4 +4,5 @@
   <xacro:arg name="prefix" default="" />
   <xacro:arg name="use_mock_hardware" default="false" />
+  <xacro:arg name="use_sim" default="true" />
   <xacro:include filename="diffbot_description.urdf.xacro" />
   <!-- Import Rviz colors -->
@@ -11,4 +12,7 @@
   <xacro:diffbot prefix="$(arg prefix)" />
   <xacro:diffbot_ros2_control
-    name="DiffBot" prefix="$(arg prefix)" use_mock_hardware="$(arg use_mock_hardware)"/>
+    name="DiffBot"
+    prefix="$(arg prefix)"
+    use_mock_hardware="$(arg use_mock_hardware)"
+    use_sim="$(arg use_sim)" />
 </robot>

File: src/differential_drive/src/description/urdf/diffbot_description.urdf.xacro (robot description, xacro)
@@ -14,4 +14,10 @@
   <xacro:property name="caster_wheel_radius" value="0.015" />
   <xacro:property name="z_offset" value="-${base_height/2}" /> <!-- Space btw top of beam and the each joint -->
+  <link name="${prefix}base_footprint"/>
+  <joint name="${prefix}base_joint" type="fixed">
+    <parent link="${prefix}base_footprint"/>
+    <child link="${prefix}base_link"/>
+    <origin xyz="0 0 0" rpy="0 0 0"/>
+  </joint>
   <!-- Base Link -->
   <link name="${prefix}base_link">
