Commit message: Increased gz velocity limit so allow turning

File: src/differential_drive/src/description/urdf/diffbot_description.urdf.xacro (robot description, xacro)
@@ -18,5 +18,5 @@
     <parent link="${prefix}base_footprint"/>
     <child link="${prefix}base_link"/>
-    <origin xyz="0 0 0" rpy="0 0 0"/>
+    <origin xyz="0 0 ${(base_height/2) + wheel_radius}" rpy="0 0 0"/>
   </joint>
   <!-- Base Link -->
@@ -25,5 +25,5 @@
       <origin xyz="0 0 0" rpy="0 0 0"/>
       <geometry>
-        <box size="${base_width} ${base_length} ${base_height}"/>
+        <sphere radius="${wheel_radius}"/>
       </geometry>
     </collision>
@@ -50,5 +50,5 @@
       <axis xyz="0 1 0"/>
       <dynamics damping="0.2"/>
-      <limit effort="100" velocity="1.0"/>
+      <limit effort="100" velocity="100.0"/>
     </joint>
     <!-- left wheel Link -->
@@ -164,6 +164,29 @@
           iyy="${caster_wheel_mass * 0.4 * (caster_wheel_radius * caster_wheel_radius)}" iyz="0.0"
           izz="${caster_wheel_mass * 0.4 * (caster_wheel_radius * caster_wheel_radius)}"/>
-        </inertial>
-      </link>
+      </inertial>
+    </link>
+    <gazebo reference="${prefix}base_link">
+      <material>Gazebo/Orange</material>
+    </gazebo>
+    <gazebo reference="${prefix}left_wheel">
+      <material>Gazebo/Black</material>
+      <mu1>1.0</mu1>
+      <mu2>1.0</mu2>
+    </gazebo>
+    <gazebo reference="${prefix}right_wheel">
+      <material>Gazebo/Black</material>
+      <mu1>1.0</mu1>
+      <mu2>1.0</mu2>
+    </gazebo>
+    <gazebo reference="${prefix}caster_frontal_wheel">
+      <material>Gazebo/White</material>
+      <mu1>0.0</mu1>
+      <mu2>0.0</mu2>
+    </gazebo>
+    <gazebo reference="${prefix}caster_rear_wheel">
+      <material>Gazebo/White</material>
+      <mu1>0.0</mu1>
+      <mu2>0.0</mu2>
+    </gazebo>
   </xacro:macro>
 </robot>
