Commit message: Added color to wheels

File: src/larry_description/urdf/larry_wheels.xacro (robot description, xacro)
@@ -1,4 +1,7 @@
 <?xml version="1.0"?>
 <robot xmlns:xacro="http://www.ros.org/wiki/xacro">
+    <material name="black">
+        <color rgba="0.1 0.1 0.1 1.0"/>
+    </material>
     <xacro:macro name="build_wheel" params="prefix x y z">
         <link name="${prefix}_wheel_link">
