Commit message: Implemented gazebo launch

File: src/larry_description/urdf/larry_core.xacro (robot description, xacro)
@@ -6,5 +6,5 @@
             <parent link="base_link"/>
             <child link="part_1"/>
-            <origin xyz="0 0 0" rpy="0 0 0"/>
+            <origin xyz="0 0 0.41" rpy="0 0 0"/>
         </joint>
         <!-- Link part_1 -->
