Commit message: Added ros2_control joints

File: src/larry_description/urdf/larry.ros2_control.xacro (robot description, xacro)
@@ -8,5 +8,47 @@
                 </xacro:if>
             </hardware>
+            <!-- left_wheel_names -->
             <joint name="front_left_wheel_joint">
+                <command_interface name="velocity">
+                    <param name="min">-10</param>
+                    <param name="max">10</param>
+                </command_interface>
+                <state_interface name="position"/>
+                <state_interface name="velocity"/>
+            </joint>
+            <joint name="mid_left_wheel_joint">
+                <command_interface name="velocity">
+                    <param name="min">-10</param>
+                    <param name="max">10</param>
+                </command_interface>
+                <state_interface name="position"/>
+                <state_interface name="velocity"/>
+            </joint>
+            <joint name="rear_left_wheel_joint">
+                <command_interface name="velocity">
+                    <param name="min">-10</param>
+                    <param name="max">10</param>
+                </command_interface>
+                <state_interface name="position"/>
+                <state_interface name="velocity"/>
+            </joint>
+            <!-- right_wheel_names -->
+            <joint name="front_right_wheel_joint">
+                <command_interface name="velocity">
+                    <param name="min">-10</param>
+                    <param name="max">10</param>
+                </command_interface>
+                <state_interface name="position"/>
+                <state_interface name="velocity"/>
+            </joint>
+            <joint name="mid_right_wheel_joint">
+                <command_interface name="velocity">
+                    <param name="min">-10</param>
+                    <param name="max">10</param>
+                </command_interface>
+                <state_interface name="position"/>
+                <state_interface name="velocity"/>
+            </joint>
+            <joint name="rear_right_wheel_joint">
                 <command_interface name="velocity">
                     <param name="min">-10</param>

Commit message: Schedlued nodes

File: src/larry_description/urdf/larry.ros2_control.xacro (robot description, xacro)
@@ -7,4 +7,9 @@
                     <plugin>gz_ros2_control/GazeboSimSystem</plugin>
                 </xacro:if>
+                <!-- TODO:: Implement LarrySystemHardware -->
+                <xacro:unless value="${use_sim}">
+                    <plugin>larry_hardware/LarrySystemHardware</plugin>
+                    <param name="serial_port">/dev/ttyUSB0</param>
+                </xacro:unless>
             </hardware>
             <!-- left_wheel_names -->

File: src/larry_description/urdf/larry.urdf.xacro (robot description, xacro)
@@ -3,4 +3,5 @@
   xmlns:xacro="http://www.ros.org/wiki/xacro">
   <xacro:arg name="use_sim" default="true"/>
+  <xacro:property name="use_sim_val" value="$(arg use_sim)" />
   <xacro:include filename="larry_core.xacro" />
   <xacro:include filename="larry_wheels.xacro" />
@@ -14,4 +15,4 @@
   <xacro:build_wheel prefix="rear_left" x="-0.16" y="0.33" z="-0.35" />
   <xacro:build_wheel prefix="rear_right" x="0.5" y="0.33" z="-0.35" />
-  <xacro:larry_ros2_control use_sim="$(arg use_sim)" />
+  <xacro:larry_ros2_control use_sim="${use_sim_val}" />
 </robot>
