Commit message: feat(Slam): integrate Larry robot with Gazebo SLAM simulation
- Add Slam package to .gitignore allowlist
- Move larry URDF files from larry_description/urdf to Slam/description
  (larry.urdf.xacro, larry_core.xacro, larry_wheels.xacro, larry.ros2_control.xacro)
- Remove old robot description files (face, inertial_macros, robot_core, ros2_control, robot.urdf)
- Update lidar.xacro and depth_camera.xacro to use part_1 as parent link
- Fix controllers.yaml: 6-wheel diff drive config, use_stamped_vel: true
- Fix slam_params.yaml: use base_link frame (not base_footprint)
- Fix lidar_sim_launch.py: set GZ_SIM_RESOURCE_PATH for larry_description meshes
- Update README: build command, TwistStamped cmd_vel topic, teleop instructions

Co-Authored-By: Claude Sonnet 4.6 <noreply@anthropic.com>

File: src/Slam/description/depth_camera.xacro (robot description, xacro)
@@ -2,7 +2,8 @@
 <robot xmlns:xacro="http://www.ros.org/wiki/xacro" >
     <joint name="camera_joint" type="fixed">
-        <parent link="chassis"/>
+        <parent link="part_1"/>
         <child link="camera_link"/>
-        <origin xyz="0.305 0 0.08" rpy="0 0 0"/>
+        <!-- Mounted at the front of the robot body -->
+        <origin xyz="0.17 -0.33 0.1" rpy="0 0 0"/>
     </joint>
     <link name="camera_link">
@@ -19,5 +20,5 @@
         <origin xyz="0 0 0" rpy="${-pi/2} 0 ${-pi/2}"/>
     </joint>
-    <link name="camera_link_optical"></link>
+    <link name="camera_link_optical"/>
     <gazebo reference="camera_link">
         <material>Gazebo/Red</material>

File: src/Slam/description/larry.ros2_control.xacro (robot description, xacro)
@@ -67,5 +67,5 @@
             <gazebo>
                 <plugin filename="gz_ros2_control-system" name="gz_ros2_control::GazeboSimROS2ControlPlugin">
-                    <parameters>$(find larry_description)/config/diffbot_controllers.yaml</parameters>
+                    <parameters>$(find Slam)/config/controllers.yaml</parameters>
                 </plugin>
             </gazebo>

File: src/Slam/description/larry.urdf.xacro (robot description, xacro)
@@ -7,4 +7,10 @@
   <xacro:include filename="larry_wheels.xacro" />
   <xacro:include filename="larry.ros2_control.xacro" />
+  <xacro:include filename="lidar.xacro" />
+  <xacro:include filename="depth_camera.xacro" />
+  <!-- red is used by depth_camera.xacro; black is already defined in larry_wheels.xacro -->
+  <material name="red">
+    <color rgba="0.8 0.1 0.1 1.0"/>
+  </material>
   <xacro:larry_core />
   <!-- Approximated values -->
@@ -16,3 +22,6 @@
   <xacro:build_wheel prefix="rear_right" x="0.5" y="0.33" z="-0.35" />
   <xacro:larry_ros2_control use_sim="${use_sim_val}" />
+  <!-- NOTE: gz-sim-sensors-system is NOT registered here because playground.sdf
+       already registers it at the world level. Adding it again at the model level
+       causes a duplicate renderer/scene crash (segfault in SensorsPrivate::WaitForInit). -->
 </robot>

File: src/Slam/description/lidar.xacro (robot description, xacro)
@@ -2,7 +2,8 @@
 <robot xmlns:xacro="http://www.ros.org/wiki/xacro" >
     <joint name="laser_joint" type="fixed">
-        <parent link="chassis"/>
+        <parent link="part_1"/>
         <child link="laser"/>
-        <origin xyz="0.122 0 0.212" rpy="0 0 0"/>
+        <!-- Mounted at center-top of robot body, toward the front -->
+        <origin xyz="0.17 -0.2 0.2" rpy="0 0 0"/>
     </joint>
     <!-- Match real-world driver frame_id ('laser') -->
@@ -14,11 +15,4 @@
             <material name="black"/>
         </visual>
-        <visual>
-            <origin xyz="0 0 -0.05"/>
-            <geometry>
-                <cylinder radius="0.01" length="0.1"/>
-            </geometry>
-            <material name="black"/>
-        </visual>
         <collision>
             <geometry>
@@ -26,7 +20,10 @@
             </geometry>
         </collision>
-        <xacro:inertial_cylinder mass="0.1" length="0.04" radius="0.05">
+        <inertial>
             <origin xyz="0 0 0" rpy="0 0 0"/>
-        </xacro:inertial_cylinder>
+            <mass value="0.1"/>
+            <inertia ixx="6.458e-5" ixy="0" ixz="0"
+                     iyy="6.458e-5" iyz="0" izz="9.817e-5"/>
+        </inertial>
     </link>
     <gazebo reference="laser">
@@ -36,13 +33,16 @@
             <topic>scan</topic>
             <update_rate>10</update_rate>
-            <gz_frame_id>laser</gz_frame_id> <always_on>1</always_on>
+            <gz_frame_id>laser</gz_frame_id>
+            <always_on>1</always_on>
             <visualize>true</visualize>
             <ray>
                 <scan>
                     <horizontal>
-                        <samples>360</samples> <resolution>1</resolution>
-                        <min_angle>-3.14159</min_angle> <max_angle>3.14159</max_angle>
+                        <samples>360</samples>
+                        <resolution>1</resolution>
+                        <min_angle>-3.14159</min_angle>
+                        <max_angle>3.14159</max_angle>
                     </horizontal>
-                    </scan>
+                </scan>
                 <range>
                     <min>0.1</min>
